File: headfan.sch (KiCad schematic (older format))
At the start: 14 parts

Commit message: - added charge controller - started layout
Parts:
- removed D?: red, symbol Device:LED
- added C1, C2: 1u/6V3, Capacitor_SMD:C_0805_2012Metric, symbol Device:C
- added IC1: MCP73811, Package_TO_SOT_SMD:SOT-23-5, symbol Auktoralib:MCP73811
- added J1: USB, Connector_USB:USB_Micro-B_Wuerth_629105150521, symbol Connector:USB_B_Micro
- added J2: Battery, Connector_PinHeader_2.54mm:PinHeader_1x02_P2.54mm_Horizontal, symbol Connector_Generic:Conn_01x02
- added J4: Fan, Connector_PinHeader_2.54mm:PinHeader_1x02_P2.54mm_Horizontal, symbol Connector_Generic:Conn_01x02
- C3, C4, C5, C6: renamed from C?; footprint (none) -> Capacitor_SMD:C_0805_2012Metric
- D1: renamed from D?; footprint (none) -> LED_SMD:LED_0805_2012Metric
- D2: renamed from D?; footprint (none) -> Diode_SMD:D_SOD-123
- IC2: renamed from IC?; footprint (none) -> Package_TO_SOT_SMD:SOT-23-5
- J3: renamed from J?; footprint (none) -> Connector_Samtec_HLE_SMD:Samtec_HLE-103-02-xxx-DV_2x03_P2.54mm_Horizontal
- L1: renamed from L?; value INDUCTOR -> NRS6028T101MMGJ; footprint (none) -> Inductor_SMD:L_Taiyo-Yuden_NR-60xx
- Q1: renamed from Q?; footprint (none) -> Package_TO_SOT_SMD:SOT-23
- R1, R2: renamed from R?; footprint (none) -> Resistor_SMD:R_0805_2012Metric
- U1: renamed from U?; footprint Package_SO:SOIC-8_3.9x4.9mm_P1.27mm -> Package_SO:SOIC-8_5.23x5.23mm_P1.27mm
Connections:
- wire segments 27 -> 41
